File: Kicad_PCB/board_30x15_side04/board_30x15_side04.kicad_pcb (KiCad board)
At the start: 2 copper layers, 30 x 15 mm, 2 parts

Commit message: components schema
Parts:
- added C1: 2.5uF, Capacitor_SMD:C_0805_2012Metric, F.Cu at (153.2, 135.4)
- added C2: 4.7uF, Capacitor_SMD:C_0805_2012Metric, F.Cu at (145.1, 127.3)
- added C3: 0.1uF, Capacitor_SMD:C_0805_2012Metric, F.Cu at (148.3, 126.5)
- added C4: 2.5uF, Capacitor_SMD:C_0805_2012Metric, F.Cu at (159.3, 130.5)
- added J1: Conn_01x08_Male, Connector_Hirose:Hirose_DF13-08P-1.25DSA_1x08_P1.25mm_Vertical, F.Cu at (137.5, 126.4)
- added Q1: BF545A, Package_TO_SOT_SMD:SOT-23, F.Cu at (155.8, 128.1)
- added Q2: BF545A, Package_TO_SOT_SMD:SOT-23, F.Cu at (154.9, 132.0)
- added R1: 1k, Resistor_SMD:R_0402_1005Metric, F.Cu at (149.9, 135.8)
- added R2: 10, Resistor_SMD:R_0402_1005Metric, F.Cu at (152.7, 128.3)
- added R3: 100, Resistor_SMD:R_0402_1005Metric, F.Cu at (152.7, 125.8)
- added R4: 100, Resistor_SMD:R_0402_1005Metric, F.Cu at (152.0, 131.7)
- added R5: 10, Resistor_SMD:R_0402_1005Metric, F.Cu at (160.0, 133.7)
- added R6: 1k, Resistor_SMD:R_0402_1005Metric, F.Cu at (160.2, 128.3)
- added R7: 50, Resistor_SMD:R_0402_1005Metric, F.Cu at (141.4, 133.9)
- added R8: 50, Resistor_SMD:R_0402_1005Metric, F.Cu at (141.6, 130.5)
- added U1: MC34152, Package_SO:SOIC-8_3.9x4.9mm_P1.27mm, F.Cu at (146.8, 131.3)
- L1, L2: value 400uH -> 0.4mH
Connections:
- L1 pad 1: unconnected-(L1-Pad1) -> Net-(C1-Pad1)
- L1 pad 2: unconnected-(L1-Pad2) -> GND
- L2 pad 1: unconnected-(L2-Pad1) -> Net-(C4-Pad1)
- L2 pad 2: unconnected-(L2-Pad2) -> GND

Commit message: sensor board
Parts:
- added D1: LED, LED_THT:LED_D1.8mm_W1.8mm_H2.4mm_Horizontal_O1.27mm_Z1.6mm, B.Cu at (138.6, 131.8)
- added R10: 50, Resistor_SMD:R_0402_1005Metric, F.Cu at (157.4, 129.2)
- added R9: 50, Resistor_SMD:R_0402_1005Metric, F.Cu at (145.8, 132.0)
- J1: moved to B.Cu
- moved J1 26.4 mm to (163.9, 125.8)
- moved R7 18.9 mm to (159.6, 128.8)
- moved R8 18.0 mm to (159.6, 130.4)
- moved Q1 13.7 mm to (142.6, 131.6)
- moved R3 10.6 mm to (142.4, 128.4)
- moved R1 9.44 mm to (159.2, 134.2)
- moved R2 8.49 mm to (145.9, 133.4)
- moved C4 7.78 mm to (153.0, 135.0), turned to 180 degrees
- moved Q2 6.67 mm to (151.6, 126.2), turned to 180 degrees
- moved U1 5.81 mm to (152.6, 131.0)
- moved R4 5.67 mm to (155.7, 127.4), turned to 180 degrees
- moved R6 4.55 mm to (157.4, 131.9), turned to 90 degrees
- moved C1 3.97 mm to (149.2, 135.0)
- moved C2 3.00 mm to (146.4, 130.0)
- moved C3 1.86 mm to (146.6, 127.2), turned to 180 degrees
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Connections:
- C1 pad 1: Net-(C1-Pad1) -> /fb2
- J1 pad 4: unconnected-(J1-Pad4) -> /fb1
- J1 pad 5: unconnected-(J1-Pad5) -> /fb2
- J1 pad 6: unconnected-(J1-Pad6) -> /led1
- L1 pad 1: Net-(C1-Pad1) -> /fb2
- R1 pad 1: Net-(Q1-Pad2) -> /fb1
- R2 pad 1: Net-(Q1-Pad2) -> /fb1
- R2 pad 2: Net-(C1-Pad1) -> /fb2
- R5 pad 2: Net-(Q2-Pad2) -> Net-(R10-Pad2)
- R6 pad 1: Net-(Q2-Pad2) -> Net-(R10-Pad2)
