File: Kicad_PCB/board_30x15_side04/board_30x15_side04.kicad_sch (KiCad schematic)
At the start: 2 parts

Commit message: components schema
Parts:
- added C1, C4: 2.5uF, Capacitor_SMD:C_0805_2012Metric, symbol Device:C
- added C2: 4.7uF, Capacitor_SMD:C_0805_2012Metric, symbol Device:C
- added C3: 0.1uF, Capacitor_SMD:C_0805_2012Metric, symbol Device:C
- added J1: Conn_01x08_Male, Connector_Hirose:Hirose_DF13-08P-1.25DSA_1x08_P1.25mm_Vertical, symbol Connector:Conn_01x08_Male
- added Q1, Q2: BF545A, Package_TO_SOT_SMD:SOT-23, symbol Transistor_FET:BF545A
- added R1, R6: 1k, Resistor_SMD:R_0402_1005Metric, symbol Device:R
- added R2, R5: 10, Resistor_SMD:R_0402_1005Metric, symbol Device:R
- added R3, R4: 100, Resistor_SMD:R_0402_1005Metric, symbol Device:R
- added R7, R8: 50, Resistor_SMD:R_0402_1005Metric, symbol Device:R
- added U1: MC34152, Package_SO:SOIC-8_3.9x4.9mm_P1.27mm, symbol Driver_FET:MC34152
- L1, L2: value 400uH -> 0.4mH
Connections:
- net at L1.1: now also C1.1, R2.2
- net GND: now reaches L1.2
- net GND: now also L2.2, C1.2, C2.1, C3.2, C4.2, J1.8 (Pin_8), R1.2, R6.2, R7.2, R8.2, U1.3 (GND)
- net at L2.1: now also C4.1, R5.1
- new net: R3.1, U1.5 (OUT_B)
- new net: Q1.2 (D), R1.1, R2.1
- new net: Q2.2 (D), R5.2, R6.1
- new net: Q2.3 (G), R4.1
- new net: R4.2, U1.7 (OUT_A)
- new net: J1.2 (Pin_2), R7.1, U1.2 (IN_A)
- new net: J1.3 (Pin_3), R8.1, U1.4 (IN_B)
- new net VCC: C2.2, C3.1, J1.1 (Pin_1), Q1.1 (S), Q2.1 (S), U1.6 (V+)
- new net out_B: Q1.3 (G), R3.2

Commit message: sensor board
Parts:
- added D1: LED, LED_THT:LED_D1.8mm_W1.8mm_H2.4mm_Horizontal_O1.27mm_Z1.6mm, symbol Device:LED
- added R10, R9: 50, Resistor_SMD:R_0402_1005Metric, symbol Device:R
Connections:
- net GND: now also D1.1 (K)
- net fb2: now reaches C1.1, L1.1, R2.2
- net fb2: now also J1.5 (Pin_5)
- net fb1: now reaches R1.1, R2.1
- net fb1: now also J1.4 (Pin_4), R9.2; no longer Q1.2 (D)
- net at R5.2, R6.1: now also R10.2; no longer Q2.2 (D)
- net led1: now reaches J1.6 (Pin_6)
- net led1: now also D1.2 (A)
- new net: Q1.2 (D), R9.1
- new net: Q2.2 (D), R10.1
Other:
- moved on the sheet: R2
